File: projects/06-shift_register/circuit/shift_register.kicad_sch (KiCad schematic)
At the start: 5 parts, among them SW2 SW_MEC_5E

Commit message: FEAT add the circuit shemma to the circuit folder
Parts:
- removed SW2: SW_MEC_5E, symbol Switch:SW_MEC_5E
- added D2, D3, D4, D5, D6, D7, D8: LED, symbol Device:LED
- added R3, R4, R5, R6, R7, R8: 220, symbol Device:R
- added U1: 74HC595, symbol 74xx:74HC595
- R1, R2: value 10000 -> 220
Connections:
- net GND: now also A1.29 (GND), R3.2, R4.2, R5.2, R6.2, R7.2, R8.2; no longer A1.6 (GND)
- net at R2.1: now also D2.1 (K)
- net at A1.25 (D10): no longer D1.2 (A)
- net at A1.5 (+5V): now also U1.10 (~{SRCLR}), U1.16 (VCC)
- net at A1.23 (D8): now also U1.12 (RCLK)
- net at A1.26 (D11): now also U1.14 (SER)
- net at A1.28 (D13): now also U1.11 (SRCLK)
- new net: D5.1 (K), R5.1
- new net: D4.1 (K), R4.1
- new net: D4.2 (A), U1.3 (QD)
- new net: D8.1 (K), R8.1
- new net: D3.1 (K), R3.1
- new net: D6.1 (K), R6.1
- new net: D7.1 (K), R7.1
- new net: D5.2 (A), U1.4 (QE)
- new net: A1.6 (GND), U1.13 (~{OE}), U1.8 (GND)
- new net: D2.2 (A), U1.1 (QB)
- new net: D1.2 (A), U1.15 (QA)
- new net: D8.2 (A), U1.7 (QH)
- new net: D7.2 (A), U1.6 (QG)
- new net: D3.2 (A), U1.2 (QC)
- new net: D6.2 (A), U1.5 (QF)
